File: schematic/desk-schematic.sch (KiCad schematic (older format))
At the start: 6 parts, among them SW1 SW_DIP_x01, U1 WeMos_D1_mini

Commit message: feat(schematic): Redo schematic to new design
Parts:
- removed DeskConnector1, SwitchConnector1: DIN-7, symbol Connector:DIN-7
- removed SW1: SW_DIP_x01, symbol Switch:SW_DIP_x01
- added ButtonConnector1, DeskConnector1: DIN-7-GND, Connector_JST:JST_XH_B8B-XH-AM_1x08_P2.50mm_Vertical, symbol desk:DIN-7-GND
- added D1, D2: D, Diode_THT:D_DO-34_SOD68_P7.62mm_Horizontal, symbol Device:D
- added J1: Conn_01x09, Connector_JST:JST_XH_B9B-XH-AM_1x09_P2.50mm_Vertical, symbol Connector_Generic:Conn_01x09
- added J2: Conn_01x09, symbol Connector_Generic:Conn_01x09
- added J3: Conn_01x03, Connector_JST:JST_XH_B3B-XH-AM_1x03_P2.50mm_Vertical, symbol Connector_Generic:Conn_01x03
- added J4: Conn_01x03, symbol Connector_Generic:Conn_01x03
- added R1, R2, R3, R4: R, Resistor_THT:R_Axial_DIN0204_L3.6mm_D1.6mm_P7.62mm_Horizontal, symbol Device:R
- added SW1: SW_3PDT, symbol desk:SW_3PDT
- added SW2: SW_DIP_x01, Button_Switch_THT:SW_DIP_SPSTx01_Slide_9.78x4.72mm_W7.62mm_P2.54mm, symbol Switch:SW_DIP_x01
Connections:
- net labels added: 5V_SWITCHED, ASSERT_DOWN, ASSERT_UP, BTN_DOWN, BTN_UP, CTL_DOWN, CTL_UP, LV_CTL_DOWN, LV_CTL_UP, PowerLED, StatusLED
- net labels removed: HS1, HS2, POWER_LED, STATUS_LED
- wire segments 2 -> 88
- no-connect marks 0 -> 9
Other:
- note added: "1: Brown RxD\n2: Blue HS3\n3: Green HS1 Button up\n4: Yellow HS4\n5: White HS2 Button Down\n6: Orange TxD\n7: Red 5v\n8/shell: Black gnd"
- note removed: "DIN shell is ground"
